File: ExoMotorBoard_v1/InputCircuit.sch (KiCad schematic (older format))
At the start: 0 parts

Commit message: Encoder connectors added in the schematic
Parts:
- added E_Front, E_Joint, E_Joint_Out, E_Rear: Conn_01x05_Male, symbol Connector:Conn_01x05_Male
Connections:
- net labels added: +5V, Front_5v, Front_A, Front_B, Front_G, Front_I, GND, Joint_5v, Joint_A, Joint_B, Joint_G, Joint_I, Rear_5v, Rear_A, Rear_B, Rear_G, Rear_I
- wire segments 0 -> 20
Other:
- note added: "Encoder Input terminals\n"
- note added: "Encoder Output Terminal\n"
Changed lines of the file:
@@
 $Descr A4 11693 8268
 encoding utf-8
-Sheet 1 8
+Sheet 2 8
 Title ""
 Date ""
@@
 Comment4 ""
 $EndDescr
+$Comp
+L Connector:Conn_01x05_Male E_Front
+U 1 1 6126FD94
+P 1000 1100
+F 0 "E_Front" H 1108 1481 50  0000 C CNN
+F 1 "Conn_01x05_Male" H 1108 1390 50  0000 C CNN
+F 2 "" H 1000 1100 50  0001 C CNN
+F 3 "~" H 1000 1100 50  0001 C CNN
+	1    1000 1100
+	1    0    0    -1
+$EndComp
+$Comp
+L Connector:Conn_01x05_Male E_Joint
+U 1 1 612704A3
+P 1000 1950
+F 0 "E_Joint" H 1108 2331 50  0000 C CNN
+F 1 "Conn_01x05_Male" H 1108 2240 50  0000 C CNN
+F 2 "" H 1000 1950 50  0001 C CNN
+F 3 "~" H 1000 1950 50  0001 C CNN
+	1    1000 1950
+	1    0    0    -1
+$EndComp
+$Comp
+L Connector:Conn_01x05_Male E_Rear
+U 1 1 61271073
+P 1000 2900
+F 0 "E_Rear" H 1108 3281 50  0000 C CNN
+F 1 "Conn_01x05_Male" H 1108 3190 50  0000 C CNN
+F 2 "" H 1000 2900 50  0001 C CNN
+F 3 "~" H 1000 2900 50  0001 C CNN
+	1    1000 2900
+	1    0    0    -1
+$EndComp
+Wire Wire Line
+	1200 900  1950 900
+Wire Wire Line
+	1200 1750 1950 1750
+Wire Wire Line
+	1200 1950 1950 1950
+Wire Wire Line
+	1200 2050 1950 2050
+Wire Wire Line
+	1200 2700 1950 2700
+Wire Wire Line
+	1200 2900 1950 2900
+Wire Wire Line
+	1200 3000 1950 3000
+Text Label 1600 1200 0    50   ~ 0
+Front_I
+Text Label 1600 1300 0    50   ~ 0
+Front_G
+Text Label 1600 1100 0    50   ~ 0
+Front_A
+Text Label 1600 1000 0    50   ~ 0
+Front_5v
+Wire Wire Line
+	1200 1200 1950 1200
+Wire Wire Line
+	1200 1100 1950 1100
+Text Label 1600 900  0    50   ~ 0
+Front_B
+Text Label 1600 1750 0    50   ~ 0
+Joint_B
+Text Label 1600 1850 0    50   ~ 0
+Joint_5v
+Text Label 1600 1950 0    50   ~ 0
+Joint_A
+Text Label 1600 2050 0    50   ~ 0
+Joint_I
+Text Label 1600 2150 0    50   ~ 0
+Joint_G
+Text Label 1600 2700 0    50   ~ 0
+Rear_B
+Text Label 1600 2800 0    50   ~ 0
+Rear_5v
+Text Label 1600 2900 0    50   ~ 0
+Rear_A
+Text Label 1600 3000 0    50   ~ 0
+Rear_I
+Text Label 1600 3100 0    50   ~ 0
+Rear_G
+$Comp
+L power:GND #PWR?
+U 1 1 6127BF60
+P 2350 1300
+F 0 "#PWR?" H 2350 1050 50  0001 C CNN
+F 1 "GND" V 2355 1172 50  0000 R CNN
+F 2 "" H 2350 1300 50  0001 C CNN
+F 3 "" H 2350 1300 50  0001 C CNN
+	1    2350 1300
+	0    -1   -1   0
+$EndComp
+Wire Wire Line
+	1200 1300 2350 1300
+$Comp
+L power:GND #PWR?
+U 1 1 6127C9E8
+P 2350 2150
+F 0 "#PWR?" H 2350 1900 50  0001 C CNN
+F 1 "GND" V 2355 2022 50  0000 R CNN
+F 2 "" H 2350 2150 50  0001 C CNN
+F 3 "" H 2350 2150 50  0001 C CNN
+	1    2350 2150
+	0    -1   -1   0
+$EndComp
+$Comp
+L power:GND #PWR?
+U 1 1 6127CE32
+P 2300 3100
+F 0 "#PWR?" H 2300 2850 50  0001 C CNN
+F 1 "GND" V 2305 2972 50  0000 R CNN
+F 2 "" H 2300 3100 50  0001 C CNN
+F 3 "" H 2300 3100 50  0001 C CNN
+	1    2300 3100
+	0    -1   -1   0
+$EndComp
+Wire Wire Line
+	1200 2150 2350 2150
+Wire Wire Line
+	1200 3100 2300 3100
+$Comp
+L power:+5V #PWR?
+U 1 1 6128124C
+P 2300 2800
+F 0 "#PWR?" H 2300 2650 50  0001 C CNN
+F 1 "+5V" V 2315 2928 50  0000 L CNN
+F 2 "" H 2300 2800 50  0001 C CNN
+F 3 "" H 2300 2800 50  0001 C CNN
+	1    2300 2800
+	0    1    1    0
+$EndComp
+$Comp
+L power:+5V #PWR?
+U 1 1 61281CBB
+P 2300 1850
+F 0 "#PWR?" H 2300 1700 50  0001 C CNN
+F 1 "+5V" V 2315 1978 50  0000 L CNN
+F 2 "" H 2300 1850 50  0001 C CNN
+F 3 "" H 2300 1850 50  0001 C CNN
+	1    2300 1850
+	0    1    1    0
+$EndComp
+$Comp
+L power:+5V #PWR?
+U 1 1 61282444
+P 2300 1000
+F 0 "#PWR?" H 2300 850 50  0001 C CNN
+F 1 "+5V" V 2315 1128 50  0000 L CNN
+F 2 "" H 2300 1000 50  0001 C CNN
+F 3 "" H 2300 1000 50  0001 C CNN
+	1    2300 1000
+	0    1    1    0
+$EndComp
+Wire Wire Line
+	1200 1000 2300 1000
+Wire Wire Line
+	1200 1850 2300 1850
+Wire Wire Line
+	1200 2800 2300 2800
+$Comp
+L Connector:Conn_01x05_Male E_Joint_Out
+U 1 1 6128496F
+P 4000 1200
+F 0 "E_Joint_Out" H 4200 750 50  0000 R CNN
+F 1 "Conn_01x05_Male" H 4350 850 50  0000 R CNN
+F 2 "" H 4000 1200 50  0001 C CNN
+F 3 "~" H 4000 1200 50  0001 C CNN
+	1    4000 1200
+	-1   0    0    1
+$EndComp
+Wire Wire Line
+	3800 1000 3350 1000
+Wire Wire Line
+	3800 1100 3350 1100
+Wire Wire Line
+	3800 1200 3350 1200
+Wire Wire Line
+	3800 1300 3350 1300
+Wire Wire Line
+	3800 1400 3350 1400
+Text Label 3400 1000 0    50   ~ 0
+Joint_B
+Text Label 3400 1200 0    50   ~ 0
+Joint_A
+Text Label 3400 1300 0    50   ~ 0
+Joint_I
+$Comp
+L power:GND #PWR?
+U 1 1 61287320
+P 3350 1400
+F 0 "#PWR?" H 3350 1150 50  0001 C CNN
+F 1 "GND" V 3355 1272 50  0000 R CNN
+F 2 "" H 3350 1400 50  0001 C CNN
+F 3 "" H 3350 1400 50  0001 C CNN
+	1    3350 1400
+	0    1    1    0
+$EndComp
+Wire Notes Line
+	650  650  2800 650
+Wire Notes Line
+	2800 650  2800 3350
+Wire Notes Line
+	2800 3350 650  3350
+Wire Notes Line
+	650  3350 650  650
+Wire Notes Line
+	2950 650  4400 650
+Wire Notes Line
+	4400 650  4400 1600
+Wire Notes Line
+	4400 1600 2950 1600
+Wire Notes Line
+	2950 1600 2950 650
+Text Notes 650  650  0    50   ~ 0
+Encoder Input terminals\n
+Text Notes 2950 650  0    50   ~ 0
+Encoder Output Terminal\n
 $EndSCHEMATC
